File: hardware/A4-Flight-Computer/A4-Flight-Computer.kicad_pcb (KiCad board)
At the start: 2 copper layers, 103 x 110.6 mm, 33 parts, among them J1 Conn_02x20_Odd_Even, J2 USB_C_Receptacle_USB2.0_14P, J5 DEBUG, Q1 IRLML0030, SW1 RST, SW2 BOOT, U1 STM32H523RETx, U5 PTCAN3414DR

Commit message: update with new pcb standard revision
Parts:
- removed J1: Conn_02x20_Odd_Even, LAB_PCB_Standard:LAB_PCB_With_Header
- added J3: LAB_Connector_02x20, LAB_PCB_Standard:LAB_PCB_With_Header, F.Cu at (73.1, 106.6)
Routing:
- net Net-(D4-A): track 12.3 -> 23.6 mm
- net /CAN_H: track 42.8 -> 37.9 mm
- net /CAN_L: track 52.2 -> 50.9 mm
